File: Schematics/Electronics/Laser_engraver.kicad_sch (KiCad schematic)
At the start: 16 parts, among them J1 MOT_X_SOCK_2, J2 MOT_X_SOCK_1, J3 MOT_Y_SOCK, J4 Power, J5 FinalSock, J6 MOT_Z_SOCK, U4 Pico, U5 LM7805_TO220

Commit message: Setting up the project
Parts:
- removed A1, A4: Pololu_Breakout_DRV8825, Module:Pololu_Breakout-16_15.2x20.3mm, symbol Driver_Motor:Pololu_Breakout_DRV8825
- removed D1: LED, LED_THT:LED_D5.0mm, symbol Device:LED
- removed J1: MOT_X_SOCK_2, Connector_JST:JST_PH_B4B-PH-K_1x04_P2.00mm_Vertical, symbol Connector_Generic:Conn_01x04
- removed J6: MOT_Z_SOCK, Connector_JST:JST_PH_B4B-PH-K_1x04_P2.00mm_Vertical, symbol Connector_Generic:Conn_01x04
- removed R1: 1k, Resistor_THT:R_Axial_DIN0207_L6.3mm_D2.5mm_P7.62mm_Horizontal, symbol Device:R
- removed U4: Pico, MCU_RaspberryPi_and_Boards:RPi_Pico_SMD_TH, symbol MCU_RaspberryPi_and_Boards:Pico
Connections:
- net +5V: no longer A2.12 (M2)
- net F_Z: no longer names the net of J5.4 (Pin_4)
- no-connect marks 31 -> 15

Commit message: Modifying schematics
Parts:
- removed J5: FinalSock, Connector_PinSocket_2.54mm:PinSocket_1x04_P2.54mm_Vertical, symbol Connector:Conn_01x04_Socket
- added J1: FinalX, symbol Connector_Generic:Conn_01x02
- added J5: FinalY, symbol Connector_Generic:Conn_01x02
- added R1, R2: 10k, symbol Device:R
Connections:
- net +12V: now also J1.1 (Pin_1), J5.1 (Pin_1)
- net F_X: now also J1.2 (Pin_2), R1.1
- net F_Y: now also J5.2 (Pin_2), R2.1
- net GND: now also R1.2, R2.2
- no-connect marks 15 -> 14
